File: kicad/small_board_simple/ventilator.sch (KiCad schematic (older format))
At the start: 36 parts, among them J1 PJ-202A, J2 Conn_01x02, J3 Conn_01x02, J5 Conn_01x02, J6 Conn_01x02, J7 Conn_01x02, J8 Conn_01x02, J9 Conn_01x02, Q3 IRLIZ44NPBF, Q4 IRLIZ44NPBF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

Commit message: enlarges arduino footprint pads:
Parts:
- A1: footprint Module:Arduino_UNO_R3 -> small_board_simple:Arduino_UNO_R3_large_pads
Changed lines of the file:
@@
 F 0 "A1" H 2800 2856 50  0000 C CNN
 F 1 "Arduino_UNO_R3" H 3350 1742 50  0000 C CNN
-F 2 "Module:Arduino_UNO_R3" H 2950 1800 50  0001 L CNN
+F 2 "small_board_simple:Arduino_UNO_R3_large_pads" H 2950 1800 50  0001 L CNN
 F 3 "https://www.arduino.cc/en/Main/arduinoBoardUno" H 2600 3900 50  0001 C CNN
 	1    2800 2850
